Commit message: fixed go2viper URDF and DR PD gain tuning

File: legged_gym/resources/robots/go2viper/go2_src/urdf/go2 copy.urdf (robot description, URDF)
Before this commit: robot go2_viperx, 42 links, 41 joints
Links:
- removed link vx_base_link
- removed link vx_ee_arm_link
- removed link vx_ee_gripper_link
- removed link vx_fingers_link
- removed link vx_gripper_bar_link
- removed link vx_gripper_link
- removed link vx_left_finger_link
- removed link vx_lower_forearm_link
- removed link vx_right_finger_link
- removed link vx_shoulder_link
- removed link vx_upper_arm_link
- removed link vx_upper_forearm_link
- removed link vx_wrist_link
- link FL_calflower: mass 0.01 -> None
- link FL_calflower1: mass 0.01 -> None
- link FR_calflower: mass 0.01 -> None
- link FR_calflower1: mass 0.01 -> None
- link RL_calflower: mass 0.01 -> None
- link RL_calflower1: mass 0.01 -> None
- link RR_calflower: mass 0.01 -> None
- link RR_calflower1: mass 0.01 -> None
- link imu: mass 0.01 -> 0
- link radar: mass 0.01 -> 0
Joints:
- removed joint go2_to_vx_mount
- removed joint vx_ee_arm
- removed joint vx_ee_bar
- removed joint vx_ee_gripper
- removed joint vx_elbow
- removed joint vx_forearm_roll
- removed joint vx_gripper_bar
- removed joint vx_left_finger
- removed joint vx_right_finger
- removed joint vx_shoulder
- removed joint vx_waist
- removed joint vx_wrist_angle
- removed joint vx_wrist_rotate

File: legged_gym/resources/robots/go2viper/viper_src/vx300s_description/urdf/vx300s_flat_raw.urdf (robot description, URDF)
Before this commit: robot vx300s, 14 links, 13 joints
Links:
- removed link vx_base_link
- removed link vx_shoulder_link
- added link vx/base_link, mass 0.969034; collision mesh filename=meshes/interbotix/vx300s_meshes/vx300s_1_base.stl scale=0.001 0.001 0.001; visual mesh filename=meshes/interbotix/vx300s_meshes/vx300s_1_base.stl scale=0.001 0.001 0.001
- added link vx/shoulder_link, mass 0.798614; collision mesh filename=meshes/interbotix/vx300s_meshes/vx300s_2_shoulder.stl scale=0.001 0.001 0.001; visual mesh filename=meshes/interbotix/vx300s_meshes/vx300s_2_shoulder.stl scale=0.001 0.001 0.001
- link vx_gripper_bar_link: geometry collision mesh filename=meshes/interbotix/vx300s_meshes/vx300s_9_gripper_bar.stl scale=0.001 0.001 0.001; visual mesh filename=meshes/interbotix/vx300s_meshes/vx300s_9_gripper_bar.stl scale=0.001 0.001 0.001
- link vx_gripper_link: geometry collision mesh filename=meshes/interbotix/vx300s_meshes/vx300s_7_gripper.stl scale=0.001 0.001 0.001; visual mesh filename=meshes/interbotix/vx300s_meshes/vx300s_7_gripper.stl scale=0.001 0.001 0.001
- link vx_left_finger_link: geometry collision mesh filename=meshes/interbotix/vx300s_meshes/vx300s_10_gripper_finger.stl scale=0.001 0.001 0.001; visual mesh filename=meshes/interbotix/vx300s_meshes/vx300s_10_gripper_finger.stl scale=0.001 0.001 0.001
- link vx_lower_forearm_link: geometry collision mesh filename=meshes/interbotix/vx300s_meshes/vx300s_5_lower_forearm.stl scale=0.001 0.001 0.001; visual mesh filename=meshes/interbotix/vx300s_meshes/vx300s_5_lower_forearm.stl scale=0.001 0.001 0.001
- link vx_right_finger_link: geometry collision mesh filename=meshes/interbotix/vx300s_meshes/vx300s_10_gripper_finger.stl scale=0.001 0.001 0.001; visual mesh filename=meshes/interbotix/vx300s_meshes/vx300s_10_gripper_finger.stl scale=0.001 0.001 0.001
- link vx_upper_arm_link: geometry collision mesh filename=meshes/interbotix/vx300s_meshes/vx300s_3_upper_arm.stl scale=0.001 0.001 0.001; visual mesh filename=meshes/interbotix/vx300s_meshes/vx300s_3_upper_arm.stl scale=0.001 0.001 0.001
- link vx_upper_forearm_link: geometry collision mesh filename=meshes/interbotix/vx300s_meshes/vx300s_4_upper_forearm.stl scale=0.001 0.001 0.001; visual mesh filename=meshes/interbotix/vx300s_meshes/vx300s_4_upper_forearm.stl scale=0.001 0.001 0.001
- link vx_wrist_link: geometry collision mesh filename=meshes/interbotix/vx300s_meshes/vx300s_6_wrist.stl scale=0.001 0.001 0.001; visual mesh filename=meshes/interbotix/vx300s_meshes/vx300s_6_wrist.stl scale=0.001 0.001 0.001
Joints:
- added joint viper_mount: type fixed, parent base, child vx/base_link, origin xyz=0.03 0 0.057 rpy=0 0 0
- joint vx_shoulder: child vx_upper_arm_link -> vx/upper_arm_link; parent vx_shoulder_link -> vx/shoulder_link
- joint vx_waist: child vx_shoulder_link -> vx/shoulder_link; limit lower=-3.141582653589793 upper=3.141582653589793 effort=10 velocity=3.141592653589793 -> effort=10 velocity=3.141592653589793; parent vx_base_link -> vx/base_link
